File: driverconn.kicad_sch (KiCad schematic)
At the start: 3 parts, among them J1 Motor 1, J6 Motor 2, J7 395026004

Commit message: rev2
Parts:
- renumbered J1 to J3, J6 to J4, J7 to J5
Other:
- moved on the sheet: J3, J4, J5
