File: motorconn.kicad_sch (KiCad schematic)
At the start: 1 part, among them J8 395021010

Commit message: rev2
Parts:
- removed J8: 395021010, MOLEX:CONN_SD-39502-001_10P_MOL, symbol 2026-03-10_14-18-01:395021010
- added J1: Conn_02x05_Counter_Clockwise, footprints:DMC 1,5 5-G1-3,5 P20THR, symbol Connector_Generic:Conn_02x05_Counter_Clockwise
- added R1: 10k, Resistor_SMD:R_0603_1608Metric_Pad0.98x0.95mm_HandSolder, symbol Device:R
Connections:
- net 5V: now also J1.9 (Pin_9), R1.1
- net GND: now also J1.8 (Pin_8)
- net LimitIN.End: now also J1.10 (Pin_10)
- net LimitIN.Home: now also J1.1 (Pin_1)
- net Phase.A+: now also J1.7 (Pin_7)
- net Phase.A-: now also J1.6 (Pin_6)
- net Phase.B+: now also J1.5 (Pin_5)
- net Phase.B-: now also J1.4 (Pin_4)
- net VCC: now also J1.3 (Pin_3)
- new net: J1.2 (Pin_2), R1.2
