File: psu.kicad_sch (KiCad schematic)
At the start: 8 parts, among them J2 V IN, J3 V OUT, U1 XL1509-5.0

Commit message: rev2
Parts:
- removed C3: 1u, Capacitor_SMD:C_0603_1608Metric_Pad1.08x0.95mm_HandSolder, symbol Device:C
- removed C4: 470u, Capacitor_SMD:CP_Elec_8x10, symbol Device:C_Polarized
- removed C5: 180u, Capacitor_SMD:CP_Elec_8x10, symbol Device:C_Polarized
- removed D2: SS34, Diode_THT:D_DO-201AD_P3.81mm_Vertical_KathodeUp, symbol Diode:SS34
- removed J3: V OUT, MOLEX:CONN_SD-39502-001_03P_MOL, symbol 2026-03-10_14-25-05:395026003
- removed L1: 68uH/2A, Inductor_SMD:L_12x12mm_H6mm, symbol Device:L
- removed U1: XL1509-5.0, Package_SO:SOIC-8_3.9x4.9mm_P1.27mm, symbol Regulator_Switching:XL1509-5.0
- added C1, C2: 1u, Capacitor_SMD:C_0603_1608Metric_Pad1.08x0.95mm_HandSolder, symbol Device:C
Connections:
- net 5V: now also C2.2
- net GND: now also C1.2, C2.1
- net VCC: now also C1.1
Other:
- moved on the sheet: J2
