File: untitled.kicad_sch (KiCad schematic)
At the start: 27 parts, among them Q1 2N7002H, Q2 2N7002H, Q3 2N7002H, Q4 2N7002H, SW1 SW_DPST_x2

Commit message: rev2
Parts:
- removed D10, D12, D4, D5: SMAJ26CA, Diode_SMD:D_SMA, symbol Diode:SMAJ26CA
- added D1, D10, D2, D5, D6, D9: PTVS26VZ1USK, Diode_SMD:Nexperia_DSN1608-2_1.6x0.8mm, symbol Diode:PTVS26VZ1USK
- R10: renamed from R21; value 2k5 -> 4k3
- R11: renamed from R23; value 2k5 -> 4k3
- renumbered C2 to C3, C1 to C4, D1 to D4, D14 to D7, D16 to D8, Q3 to Q1, Q4 to Q2, Q1 to Q3, Q2 to Q4, R4 to R13, R5 to R2, R6 to R3, R9 to R4, R1 to R5, R10 to R6, R2 to R7, R3 to R8, R11 to R9
Connections:
- net EndExtPullup: now also D2.1 (K)
- net GND: now also D1.2 (A), D10.2 (A), D2.2 (A), D5.2 (A), D6.2 (A), D9.2 (A)
- net HomeExtPullup: now also D1.1 (K)
- net LimitIN.End: now also D5.1 (K)
- net LimitIN.Home: now also D6.1 (K)
- net LimitOUT.End: now also D10.1 (K)
- net LimitOUT.Home: now also D9.1 (K)
